File: so_26_eps_pcb/_autosave-so_26_eps_pcb.kicad_pcb (KiCad board)
At the start: 4 copper layers, 90.2 x 95.9 mm, 47 parts, among them J1 Conn_02x12_Odd_Even, J3 Conn_01x02, SW1 SW_SPDT, U1 LM22679TJ-ADJ/NOPB, U2 LM22679TJ-ADJ/NOPB

Commit message: Made some last changes to the tracing
Routing:
- net +10V_ALT: track 90.0 -> 91.3 mm
Changed lines of the file:
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@@
-	)
-	(segment
-		(start 129.54 74.491)
-		(end 129.54 47.694)
-		(width 1)
-		(layer "F.Cu")
-		(net 11)
-	)
-	(segment
-		(start 129.54 47.694)
-		(end 127 45.154)
-		(width 1)
-		(layer "F.Cu")
-		(net 11)
 	)
 	(segment
 		(start 141.097 86.048)
-		(end 129.54 74.491)
-		(width 1)
-		(layer "F.Cu")
-		(net 11)
-	)
-	(segment
-		(start 127 45.154)
+		(end 131.572 76.523)
+		(width 1)
+		(layer "F.Cu")
+		(net 11)
+	)
+	(segment
+		(start 131.572 61.664)
+		(end 127 57.092)
+		(width 1)
+		(layer "F.Cu")
+		(net 11)
+	)
+	(segment
+		(start 127 57.092)
 		(end 127 44.773)
+		(width 1)
+		(layer "F.Cu")
+		(net 11)
+	)
+	(segment
+		(start 131.572 76.523)
+		(end 131.572 61.664)
 		(width 1)
 		(layer "F.Cu")
@@
 	)
 	(segment
-		(start 131.191 87.572)
-		(end 130.683 87.572)
-		(width 1)
-		(layer "F.Cu")
-		(net 14)
-	)
-	(segment
-		(start 130.683 87.572)
-		(end 96.139 53.028)
-		(width 1)
-		(layer "F.Cu")
-		(net 14)
-	)
-	(segment
-		(start 96.139 53.028)
-		(end 96.139 42.487)
+		(start 102.108 61.283)
+		(end 104.902 61.283)
+		(width 1)
+		(layer "F.Cu")
+		(net 14)
+	)
+	(segment
+		(start 104.902 61.283)
+		(end 131.191 87.572)
+		(width 1)
+		(layer "F.Cu")
+		(net 14)
+	)
+	(segment
+		(start 96.139 42.487)
+		(end 96.139 55.314)
+		(width 1)
+		(layer "F.Cu")
+		(net 14)
+	)
+	(segment
+		(start 96.139 55.314)
+		(end 102.108 61.283)
 		(width 1)
 		(layer "F.Cu")
@@
 	)
 	(segment
-		(start 143.764 89.858)
-		(end 143.764 82.873)
-		(width 2)
-		(layer "F.Cu")
-		(net 25)
-	)
-	(segment
-		(start 137.183 77.054)
+		(start 137.656 107.257)
+		(end 137.656 95.942)
+		(width 2)
+		(layer "F.Cu")
+		(net 25)
+	)
+	(segment
+		(start 137.183 76.673)
 		(end 137.183 44.542)
 		(width 2)
@@
 	)
 	(segment
-		(start 143.891 82.746)
-		(end 138.199 77.054)
+		(start 126.998 34.357)
+		(end 118.356 34.357)
 		(width 2)
 		(layer "F.Cu")
@@
 	)
 	(segment
-		(start 137.656 107.257)
-		(end 137.656 95.942)
-		(width 2)
-		(layer "F.Cu")
-		(net 25)
-	)
-	(segment
-		(start 143.764 82.873)
-		(end 143.891 82.746)
-		(width 2)
-		(layer "F.Cu")
-		(net 25)
-	)
-	(segment
-		(start 138.199 77.054)
-		(end 137.183 77.054)
-		(width 2)
-		(layer "F.Cu")
-		(net 25)
-	)
-	(segment
-		(start 126.748 34.357)
-		(end 118.356 34.357)
-		(width 2)
-		(layer "F.Cu")
-		(net 25)
-	)
-	(segment
-		(start 137.656 95.942)
-		(end 137.541 95.827)
-		(width 2)
-		(layer "F.Cu")
-		(net 25)
-	)
-	(segment
 		(start 137.183 44.542)
-		(end 126.873 34.232)
-		(width 2)
-		(layer "F.Cu")
-		(net 25)
-	)
-	(segment
-		(start 126.873 34.232)
-		(end 126.748 34.357)
+		(end 126.998 34.357)
+		(width 2)
+		(layer "F.Cu")
+		(net 25)
+	)
+	(segment
+		(start 144.78 84.27)
+		(end 137.183 76.673)
+		(width 2)
+		(layer "F.Cu")
+		(net 25)
+	)
+	(segment
+		(start 144.78 88.842)
+		(end 144.78 84.27)
 		(width 2)
 		(layer "F.Cu")
@@
 	(segment
 		(start 137.68 95.942)
-		(end 143.764 89.858)
-		(width 2)
-		(layer "F.Cu")
+		(end 144.78 88.842)
+		(width 2)
+		(layer "F.Cu")
